File: hw/mouse.sch (KiCad schematic (older format))
At the start: 27 parts, among them J1 JUMPER2, J2 JUMPER2, J3 CONN-ISP-6, J4 CONN_2X1, J5 CONN_5X1, J6 CONN_3X1, J7 Mini-DIN-6, J8 CONN_4X2, J9 CONN_5X2, U1 12MHz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

Commit message: Initial version of PCB layout (still work in progress)
Parts:
- C1: footprint Capacitors_THT:C_RM5.08mm_5x5mm -> Capacitors_THT:C_RM5.08mm_5x2.5mm
- J7: symbol connectors:Mini-DIN-6 -> mouse-rescue:Mini-DIN-6-connectors
- U2: footprint Package_DIP:DIP-20_W7.62mm -> Housings_DIP:DIP20; symbol ics_controller_atmel:ATtiny2313-20PU -> mouse-rescue:ATtiny2313-20PU-ics_controller_atmel
Changed lines of the file:
@@
 EESchema Schematic File Version 4
-EELAYER 30 0
+LIBS:mouse-cache
+EELAYER 26 0
 EELAYER END
 $Descr A4 11693 8268
@@
 $EndDescr
 $Comp
-L connectors:Mini-DIN-6 J7
+L mouse-rescue:Mini-DIN-6-connectors J7
 U 1 1 60A5670F
 P 8900 3350
@@
 $EndComp
 $Comp
-L ics_controller_atmel:ATtiny2313-20PU U2
+L mouse-rescue:ATtiny2313-20PU-ics_controller_atmel U2
 U 1 1 60A609EE
 P 3050 5250
 F 0 "U2" H 2600 6300 50  0000 C CNN
 F 1 "ATtiny2313-20PU" H 3050 5250 50  0000 C CNN
-F 2 "Package_DIP:DIP-20_W7.62mm" H 3050 5250 50  0001 C CIN
+F 2 "Housings_DIP:DIP20" H 3050 5250 50  0001 C CIN
 F 3 "http://ww1.microchip.com/downloads/en/DeviceDoc/Atmel-2543-AVR-ATtiny2313_Datasheet.pdf" H 3050 5250 50  0001 C CNN
 	1    3050 5250
@@
 F 0 "C1" H 1400 4690 50  0000 C CNN
 F 1 "4,7nF" H 1400 4599 50  0000 C CNN
-F 2 "Capacitors_THT:C_RM5.08mm_5x5mm" H 1400 4450 60  0001 C CNN
+F 2 "Capacitors_THT:C_RM5.08mm_5x2.5mm" H 1400 4450 60  0001 C CNN
 F 3 "" H 1400 4450 60  0000 C CNN
 	1    1400 4450
@@
 Wire Bus Line
 	7800 3650 5800 3650
+Connection ~ 7800 3650
 Wire Bus Line
 	9550 3350 9550 3650
@@
 Wire Bus Line
 	8300 5200 8300 6250
-Connection ~ 7800 3650
 $EndSCHEMATC

Commit message: add Kicad PCB
Parts:
- J7: footprint (none) -> Connector_Miscelleaneus:MiniDIN_6pole; symbol mouse-rescue:Mini-DIN-6-connectors -> mouse-rescue:Mini-DIN-6-connectors-mouse-rescue
- U2: symbol mouse-rescue:ATtiny2313-20PU-ics_controller_atmel -> mouse-rescue:ATtiny2313-20PU-ics_controller_atmel-mouse-rescue
Changed lines of the file:
@@
 EESchema Schematic File Version 4
-LIBS:mouse-cache
-EELAYER 26 0
+EELAYER 30 0
 EELAYER END
 $Descr A4 11693 8268
@@
 $EndDescr
 $Comp
-L mouse-rescue:Mini-DIN-6-connectors J7
+L mouse-rescue:Mini-DIN-6-connectors-mouse-rescue J7
 U 1 1 60A5670F
 P 8900 3350
 F 0 "J7" H 8900 3717 50  0000 C CNN
 F 1 "Mini-DIN-6" H 8900 3626 50  0000 C CNN
-F 2 "" H 8900 3350 50  0001 C CNN
+F 2 "Connector_Miscelleaneus:MiniDIN_6pole" H 8900 3350 50  0001 C CNN
 F 3 "http://service.powerdynamics.com/ec/Catalog17/Section%2011.pdf" H 8900 3350 50  0001 C CNN
 	1    8900 3350
@@
 $EndComp
 $Comp
-L mouse-rescue:ATtiny2313-20PU-ics_controller_atmel U2
+L mouse-rescue:ATtiny2313-20PU-ics_controller_atmel-mouse-rescue U2
 U 1 1 60A609EE
 P 3050 5250
